Commit message: URDF loading works (without frame transformations which are not supposed to be done here)

File: src/myviz/pi_robot.urdf (robot description, URDF)
Before this commit: robot pi_robot, 3 links, 2 joints
Links:
- removed link base_link
- added link map; visual box size=0.32 0.26 0.22
Joints:
- joint neck_joint: limit (none) -> lower=-1.57 upper=1.57 effort=1 velocity=3; type fixed -> revolute
- joint torso_joint: parent base_link -> map
